File: pcb/clock-base-7seg/clock-base-7seg.kicad_pcb (KiCad board)
At the start: 2 copper layers, 118 parts, among them J1 LEDs

Commit message: update pcb
Parts:
- removed REF**: MountingHole_3.2mm_M3, MountingHole:MountingHole_3.2mm_M3
- J1: moved to B.Cu
- moved D51 230.9 mm to (245.2, 38.4)
- moved D50 215.4 mm to (232.1, 25.4), turned to 90 degrees
- moved C15 213.7 mm to (245.2, 33.2)
- moved D55 208.5 mm to (245.1, 78.1)
- moved C42 203.4 mm to (245.2, 46.4)
- moved C29 202.6 mm to (227.0, 25.5), turned to 90 degrees
- moved C55 198.5 mm to (245.2, 73.0)
- moved D52 197.6 mm to (245.1, 51.7)
- moved D49 194.3 mm to (218.7, 25.4), turned to 90 degrees
- moved D56 190.6 mm to (245.2, 91.4)
- moved C37 186.8 mm to (213.5, 25.5), turned to 90 degrees
- moved D54 178.6 mm to (218.7, 65.0), turned to 270 degrees
- moved C3 174.7 mm to (191.2, 33.0)
- moved C4 173.9 mm to (237.2, 65.0), turned to 270 degrees
- moved C46 173.4 mm to (151.5, 43.5), turned to 180 degrees
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Routing:
- net +5V: track 0.00 -> 1554.8 mm, vias 0 -> 7
- net Net-(D30-Pad2): track 0.00 -> 77.8 mm
- net Net-(D28-Pad2): track 0.00 -> 72.4 mm
- net Net-(D44-Pad2): track 0.00 -> 71.4 mm
- net Net-(D14-Pad2): track 0.00 -> 69.9 mm
- net Net-(D10-Pad2): track 0.00 -> 47.1 mm
- net Net-(D40-Pad2): track 0.00 -> 46.5 mm
- net Net-(D54-Pad2): track 0.00 -> 46.1 mm
- net Net-(D24-Pad2): track 0.00 -> 45.7 mm
- net DIN: track 0.00 -> 35.4 mm, vias 0 -> 2
- net Net-(D29-Pad2): track 0.00 -> 34.8 mm
- net Net-(D2-Pad2): track 0.00 -> 25.9 mm
- net Net-(D46-Pad2): track 0.00 -> 25.7 mm
- net Net-(D16-Pad2): track 0.00 -> 25.7 mm
- net Net-(D32-Pad2): track 0.00 -> 25.3 mm
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- added copper zone on F.Cu, net GND
Other:
- board outline added: 248 x 105 mm

Commit message: finalize pcb
Parts:
- added J2: power, Connector_PinHeader_2.54mm:PinHeader_1x02_P2.54mm_Vertical, B.Cu at (224.2, 49.8)
- moved J1 0.35 mm to (53.8, 77.0)
Routing:
- net GND: track 0.00 -> 246.2 mm, vias 0 -> 7
- net +5V: track 1554.8 -> 1596.1 mm
- net DIN: track 35.4 -> 44.7 mm, vias 2 -> 1
Other:
- board text added: "+5V"
- board text added: "DIN"
- board text added: "GND"
