File: pcb/clock-base-7seg/clock-base-7seg.sch (KiCad schematic (older format))
At the start: 117 parts, among them J1 LEDs

Commit message: update pcb
Changed lines of the file:
@@
 Wire Wire Line
 	1000 10250 1350 10250
+Text Label 1150 10350 0    50   ~ 0
+5V
+Text Label 1200 10450 0    50   ~ 0
+GND
+Text Label 1100 10250 0    50   ~ 0
+DIN
 $EndSCHEMATC

Commit message: finalize pcb
Parts:
- added J2: power, Connector_PinHeader_2.54mm:PinHeader_1x02_P2.54mm_Vertical, symbol Connector:Conn_01x02_Female
Connections:
- net +5V: now also J2.2 (Pin_2)
- net GND: now also J2.1 (Pin_1)
Changed lines of the file:
@@
 Text Label 1100 10250 0    50   ~ 0
 DIN
+$Comp
+L Connector:Conn_01x02_Female J2
+U 1 1 6044F5CA
+P 2350 10350
+F 0 "J2" H 2242 10025 50  0000 C CNN
+F 1 "power" H 2242 10116 50  0000 C CNN
+F 2 "Connector_PinHeader_2.54mm:PinHeader_1x02_P2.54mm_Vertical" H 2350 10350 50  0001 C CNN
+F 3 "~" H 2350 10350 50  0001 C CNN
+	1    2350 10350
+	-1   0    0    1
+$EndComp
+$Comp
+L power:GND #PWR012
+U 1 1 6045044C
+P 2900 10350
+F 0 "#PWR012" H 2900 10100 50  0001 C CNN
+F 1 "GND" H 2905 10177 50  0000 C CNN
+F 2 "" H 2900 10350 50  0001 C CNN
+F 3 "" H 2900 10350 50  0001 C CNN
+	1    2900 10350
+	1    0    0    -1
+$EndComp
+$Comp
+L power:+5V #PWR011
+U 1 1 604506E3
+P 2900 10250
+F 0 "#PWR011" H 2900 10100 50  0001 C CNN
+F 1 "+5V" H 2915 10423 50  0000 C CNN
+F 2 "" H 2900 10250 50  0001 C CNN
+F 3 "" H 2900 10250 50  0001 C CNN
+	1    2900 10250
+	1    0    0    -1
+$EndComp
+Wire Wire Line
+	2550 10250 2900 10250
+Text Label 2700 10250 0    50   ~ 0
+5V
+Wire Wire Line
+	2900 10350 2550 10350
+Text Label 2700 10350 0    50   ~ 0
+GND
 $EndSCHEMATC
